File: eagle/mariokard_v1.brd (EAGLE design)
At the start: 77.4 x 86 mm, 64 parts, among them SW1 KMR2, SW2 KMR2, U1 SPX3819, U3 ATMEGA32U4, U4 L298, X1 ESP-12, Y1 16MHz

Commit message: small fixes - still WIP
Parts:
- added U$29: FTDI_POGO, digikey:FTDI_POGO
Connections:
- removed net D5: U3.31
- removed net D6: U3.27
- removed net DIRA: U4.P$7, U4.P$9
- removed net DIRB: U4.P$13, U4.P$15
- removed net PWMA: U4.P$8
- removed net PWMB: U4.P$14
- new net DIRA1: U4.P$7
- new net DIRA2: U4.P$9
- new net DIRB1: U4.P$13
- new net DIRB2: U4.P$15
- new net PWMA/D5: U3.31, U4.P$8
- new net PWMB/D6: U3.27, U4.P$14
- net GND: now also U$29.6
- net RXD_5V: now also U$29.3
- net TXD: now also U$29.2
- net VIN: now also U$29.4
Other:
- outline, holes or cut-outs redrawn

Commit message: fixed copy-paste error
Parts:
- removed U$29: FTDI_POGO, digikey:FTDI_POGO
Connections:
- net GND: no longer U$29.6
- net RXD_5V: no longer U$29.3
- net TXD: no longer U$29.2
- net VIN: no longer U$29.4
Changed lines of the file:
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@@
 <element name="C10" library="SparkFun" package="NIPPON_F80" value="100uF,25V" x="59.8398625" y="35.07231875" rot="R180"/>
 <element name="J1" library="SparkFun-Connectors" package="1X07" value="" x="40.215821875" y="81.206340625" rot="R180"/>
-<element name="U$29" library="digikey" package="FTDI_POGO" value="FTDI_POGO" x="1.56718125" y="-1.61798125"/>
 </elements>
 <signals>
@@
 <contactref element="C10" pad="-"/>
 <contactref element="J1" pad="2"/>
-<contactref element="U$29" pad="6"/>
 <wire x1="61.35741875" y1="70.0146" x2="58.75741875" y2="71.8146" width="0" layer="19" extent="1-1"/>
 <wire x1="52.35741875" y1="71.8146" x2="58.75741875" y2="71.8146" width="0" layer="19" extent="1-1"/>
@@
 <wire x1="92.15881875" y1="15.540621875" x2="71.404478125" y2="15.54898125" width="0" layer="19" extent="1-1"/>
 <wire x1="94.69881875" y1="17.340621875" x2="92.15881875" y2="15.540621875" width="0" layer="19" extent="1-1"/>
-<wire x1="7.91718125" y1="-1.61798125" x2="13.9472375" y2="21.25958125" width="0" layer="19" extent="1-1"/>
 </signal>
 <signal name="VIN">
@@
 <contactref element="D21" pad="C"/>
 <contactref element="D23" pad="C"/>
-<contactref element="U$29" pad="4"/>
 <wire x1="34.189784375" y1="52.67451875" x2="44.860096875" y2="48.64608125" width="0" layer="19" extent="1-1"/>
 <wire x1="31.832434375" y1="52.659275" x2="34.189784375" y2="52.67451875" width="0" layer="19" extent="1-1"/>
@@
 <wire x1="23.040340625" y1="21.53831875" x2="20.837003125" y2="49.0321625" width="0" layer="19" extent="1-1"/>
 <wire x1="31.18358125" y1="17.7038" x2="23.040340625" y2="21.53831875" width="0" layer="19" extent="1-16"/>
-<wire x1="2.83718125" y1="-1.61798125" x2="23.040340625" y2="21.53831875" width="0" layer="19" extent="1-1"/>
 </signal>
 <signal name="RESET">
@@
 <contactref element="X1" pad="16"/>
 <contactref element="U$19" pad="2"/>
-<contactref element="U$29" pad="2"/>
 <wire x1="36.26358125" y1="17.7038" x2="25.3041" y2="28.1644" width="0" layer="19" extent="1-16"/>
-<wire x1="-2.24281875" y1="-1.61798125" x2="25.3041" y2="28.1644" width="0" layer="19" extent="1-1"/>
 </signal>
 <signal name="RESET_5V">
@@
 <contactref element="D2" pad="C"/>
 <contactref element="U$19" pad="3"/>
-<contactref element="U$29" pad="3"/>
 <wire x1="20.294596875" y1="22.0954625" x2="33.72358125" y2="17.7038" width="0" layer="19" extent="1-16"/>
-<wire x1="0.29718125" y1="-1.61798125" x2="20.294596875" y2="22.0954625" width="0" layer="19" extent="1-1"/>
 </signal>
 <signal name="VBAT">

Commit message: v1 - still needs to be tested
Parts:
- removed CN1, CN2: (no value), adafruit:JST-PH-2-SMT-RA
- removed D1: 1n4148, microbuilder:SOD-323
- removed D9: RED, microbuilder:CHIPLED_0805_NOOUTLINE
- removed J1: (no value), SparkFun-Connectors:1X07
- removed SW1, SW2: KMR2, microbuilder:BTN_KMR2_4.6X2.8
- removed U$11: ISP_POGO, digikey:POGO_ISP
- removed U$19: FTDI_POGO, digikey:FTDI_POGO
- added COLOR_SENSOR: (no value), SparkFun-Connectors:1X07
- added FTDI: FTDI_POGO, digikey:FTDI_POGO
- added GPIO0, RESET: KMR2, microbuilder:BTN_KMR2_4.6X2.8
- added GPIO0LED: RED, microbuilder:CHIPLED_0805_NOOUTLINE
- added ISP: ISP_POGO, digikey:POGO_ISP
- added MOTOR_LEFT, MOTOR_RIGHT: (no value), adafruit:JST-PH-2-SMT-RA
- moved C9 77.1 mm to (22.0, 42.1), turned to 0 degrees
- moved R13 74.6 mm to (17.9, 29.4), turned to 0 degrees
- moved COM 70.5 mm to (67.1, 76.6)
- moved R12 70.1 mm to (26.0, 39.8), turned to 0 degrees
- moved R10 69.1 mm to (67.0, 74.5), turned to 180 degrees
- moved R9 68.0 mm to (46.5, 70.7), turned to 270 degrees
- moved R1 52.4 mm to (32.1, 13.0), turned to 180 degrees
- moved C7 51.6 mm to (51.1, 68.2), turned to 180 degrees
- moved R4 50.6 mm to (40.2, 13.0), turned to 0 degrees
- moved Z2 47.4 mm to (35.2, 12.0)
- moved R7 45.7 mm to (49.8, 31.4), turned to 0 degrees
- moved Z1 45.3 mm to (37.2, 12.0)
- moved R8 44.9 mm to (49.8, 27.6), turned to 0 degrees
- moved R6 42.6 mm to (52.0, 70.7), turned to 270 degrees
- moved PWR 41.8 mm to (37.7, 78.6), turned to 90 degrees
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Connections:
- removed net C_INT: J1.6
- removed net C_LED: J1.7
- removed net D10: U3.30
- removed net D11: U3.12
- removed net D12: U3.26
- removed net D7: U3.1
- removed net D8: U3.28
- removed net D9: U3.29
- removed net DIRA1: U4.P$7
- removed net DIRA2: U4.P$9
- removed net DIRB1: U4.P$13
- removed net DIRB2: U4.P$15
- removed net N$24: COM.C
- removed net N$34: U$4.MTN1, U$4.MTN3, Z1.2, Z2.2
- removed net N$35: U$4.GND, U$4.MTN2, U$4.MTN4
- removed net RESET_5V: D1.C
- removed net RXI: U3.20
- removed net TXO: U3.21
- new net C_INT/D7: COLOR_SENSOR.6, U3.1
- new net C_LED/D8: COLOR_SENSOR.7, U3.28
- new net DIRA1/D9: U3.29, U4.P$7
- new net DIRA2/D10: U3.30, U4.P$9
- new net DIRB1/D11: U3.12, U4.P$13
- new net DIRB2/D12: U3.26, U4.P$15
- net 3.3V: now also COLOR_SENSOR.1, COLOR_SENSOR.3, GPIO0LED.A; no longer D9.A, J1.1, J1.3
- net GND: now also COLOR_SENSOR.2, COM.C, FTDI.6, GPIO0.A, GPIO0.A', RESET.A, RESET.A', U$4.GND, U$4.MTN1, U$4.MTN2, U$4.MTN3, U$4.MTN4, Z1.2, Z2.2; no longer J1.2, SW1.A, SW1.A', SW2.A, SW2.A', U$19.6
- net GPIO0: now also GPIO0.B, GPIO0.B'; no longer SW2.B, SW2.B'
- net MISO: now also ISP.1; no longer U$11.1
- net MOSI: now also ISP.4; no longer U$11.4
- net N$11: now also GPIO0LED.C; no longer D9.C
- net N$32: now also ISP.2; no longer U$11.2
- net N$33: now also ISP.6; no longer U$11.6
- net OUT1: now also MOTOR_RIGHT.1; no longer CN1.1
- net OUT2: now also MOTOR_RIGHT.2; no longer CN1.2
- net OUT3: now also MOTOR_LEFT.2; no longer CN2.2
- net OUT4: now also MOTOR_LEFT.1; no longer CN2.1
- net RESET: now also ISP.5; no longer U$11.5
- net RESET_ESP: now also RESET.B, RESET.B'; no longer D1.A, SW1.B, SW1.B'
- net RXD: now also U3.20, X1.16; no longer X1.15
- net RXD_5V: now also FTDI.3; no longer U$19.3
- net SCK: now also ISP.3; no longer U$11.3
- net SCL: now also COLOR_SENSOR.4; no longer J1.4
- net SDA: now also COLOR_SENSOR.5; no longer J1.5
- net TXD: now also FTDI.2, U3.21, X1.15; no longer U$19.2, X1.16
- net VBAT: now also D21.C, D23.C, D3.C, D5.C, U4.P$6
- net VIN: now also FTDI.4; no longer D21.C, D23.C, D3.C, D5.C, U$19.4, U4.P$6
Routing:
- net 3.3V: track 0.00 -> 218.8 mm, vias 0 -> 9
- net VBAT: track 0.00 -> 168.5 mm, vias 0 -> 2
- net TXD: track 0.00 -> 110.1 mm, vias 0 -> 6
- net VUSB: track 0.00 -> 98.5 mm, vias 0 -> 6
- net OUT1: track 0.00 -> 92.1 mm, vias 0 -> 4
- net RD-: track 0.00 -> 83.6 mm, vias 0 -> 2
- net OUT2: track 0.00 -> 82.4 mm, vias 0 -> 4
- net SCL: track 0.00 -> 81.2 mm, vias 0 -> 1
- net RXD: track 0.00 -> 78.7 mm, vias 0 -> 2
- net SDA: track 0.00 -> 76.2 mm, vias 0 -> 1
- net C_LED/D8: track 0.00 -> 74.9 mm, vias 0 -> 1
- net RD+: track 0.00 -> 67.5 mm, vias 0 -> 2
- net PWMA/D5: track 0.00 -> 65.4 mm, vias 0 -> 2
- net DIRA1/D9: track 0.00 -> 62.0 mm, vias 0 -> 2
- net DIRA2/D10: track 0.00 -> 60.7 mm, vias 0 -> 2
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- added copper zone on layer 1, net GND
- added copper zone on layer 16, net GND
Other:
- outline, holes or cut-outs redrawn
- board text added: "07/28/2016"
- board text added: "CUT OUT"
- board text added: "Felix Heibeck"
- board text added: "Jiaojiao Xu"
- board text added: "Mariokardt v1"
- board text removed: "Groundplane"
- board text removed: "make contacts for battery"
